File: esc_v3_c1/ESC1.kicad_sch (KiCad schematic)
At the start: 39 parts, among them J1 Power, J2 Inputs, J3 Output, Q1 IRF4905, Q10 S8050, Q11 S8050, Q12 S8050, Q2 IRF4905, Q3 IRF4905, Q4 S8050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

Commit message: fix n channel driver
Connections:
- net at D6.2 (A), Q12.1 (E): now also Q9.1 (G)
- net at D5.2 (A), Q11.1 (E): now also Q8.1 (G)
- net at Q12.3 (C), R9.1: no longer Q9.1 (G)
- net at Q11.3 (C), R8.1: no longer Q8.1 (G)
- net at D4.2 (A), Q10.1 (E): now also Q7.1 (G)
- net at Q10.3 (C), R7.1: no longer Q7.1 (G)
Changed lines of the file:
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@@
   (junction (at 166.37 105.41) (diameter 0) (color 0 0 0 0)
   )
+  (junction (at 222.25 104.14) (diameter 0) (color 0 0 0 0)
+  )
   (junction (at 176.53 101.6) (diameter 0) (color 0 0 0 0)
   )
   (junction (at 231.14 105.41) (diameter 0) (color 0 0 0 0)
   )
-  (junction (at 92.71 93.98) (diameter 0) (color 0 0 0 0)
-  )
   (junction (at 222.25 63.5) (diameter 0) (color 0 0 0 0)
   )
@@
   (junction (at 113.03 74.93) (diameter 0) (color 0 0 0 0)
   )
-  (junction (at 222.25 93.98) (diameter 0) (color 0 0 0 0)
-  )
   (junction (at 231.14 74.93) (diameter 0) (color 0 0 0 0)
   )
-  (junction (at 157.48 93.98) (diameter 0) (color 0 0 0 0)
-  )
   (junction (at 102.87 105.41) (diameter 0) (color 0 0 0 0)
   )
@@
   (junction (at 176.53 86.36) (diameter 0) (color 0 0 0 0)
   )
+  (junction (at 219.71 104.14) (diameter 0) (color 0 0 0 0)
+  )
   (junction (at 241.3 101.6) (diameter 0) (color 0 0 0 0)
   )
+  (junction (at 92.71 104.14) (diameter 0) (color 0 0 0 0)
+  )
   (junction (at 113.03 88.9) (diameter 0) (color 0 0 0 0)
   )
+  (junction (at 157.48 104.14) (diameter 0) (color 0 0 0 0)
+  )
   (junction (at 166.37 74.93) (diameter 0) (color 0 0 0 0)
   )
@@
     (stroke (width 0) (type default) (color 0 0 0 0))
   )
+  (wire (pts (xy 100.33 104.14) (xy 100.33 93.98))
+    (stroke (width 0) (type default) (color 0 0 0 0))
+  )
+  (wire (pts (xy 226.06 93.98) (xy 236.22 93.98))
+    (stroke (width 0) (type default) (color 0 0 0 0))
+  )
   (wire (pts (xy 231.14 101.6) (xy 231.14 105.41))
     (stroke (width 0) (type default) (color 0 0 0 0))
@@
     (stroke (width 0) (type default) (color 0 0 0 0))
   )
+  (wire (pts (xy 92.71 104.14) (xy 100.33 104.14))
+    (stroke (width 0) (type default) (color 0 0 0 0))
+  )
   (wire (pts (xy 88.9 104.14) (xy 92.71 104.14))
     (stroke (width 0) (type default) (color 0 0 0 0))
@@
     (stroke (width 0) (type default) (color 0 0 0 0))
   )
-  (wire (pts (xy 218.44 104.14) (xy 222.25 104.14))
-    (stroke (width 0) (type default) (color 0 0 0 0))
-  )
   (wire (pts (xy 113.03 88.9) (xy 113.03 101.6))
     (stroke (width 0) (type default) (color 0 0 0 0))
@@
     (stroke (width 0) (type default) (color 0 0 0 0))
   )
+  (wire (pts (xy 100.33 93.98) (xy 107.95 93.98))
+    (stroke (width 0) (type default) (color 0 0 0 0))
+  )
   (wire (pts (xy 124.46 68.58) (xy 149.86 68.58))
     (stroke (width 0) (type default) (color 0 0 0 0))
@@
     (stroke (width 0) (type default) (color 0 0 0 0))
   )
+  (wire (pts (xy 222.25 104.14) (xy 226.06 104.14))
+    (stroke (width 0) (type default) (color 0 0 0 0))
+  )
   (wire (pts (xy 176.53 71.12) (xy 176.53 74.93))
     (stroke (width 0) (type default) (color 0 0 0 0))
@@
     (stroke (width 0) (type default) (color 0 0 0 0))
   )
-  (wire (pts (xy 222.25 93.98) (xy 236.22 93.98))
-    (stroke (width 0) (type default) (color 0 0 0 0))
-  )
-  (wire (pts (xy 171.45 93.98) (xy 157.48 93.98))
+  (wire (pts (xy 161.29 93.98) (xy 171.45 93.98))
     (stroke (width 0) (type default) (color 0 0 0 0))
   )
@@
     (stroke (width 0) (type default) (color 0 0 0 0))
   )
-  (wire (pts (xy 92.71 93.98) (xy 107.95 93.98))
-    (stroke (width 0) (type default) (color 0 0 0 0))
-  )
   (wire (pts (xy 71.12 63.5) (xy 73.66 63.5))
     (stroke (width 0) (type default) (color 0 0 0 0))
@@
     (stroke (width 0) (type default) (color 0 0 0 0))
   )
+  (wire (pts (xy 200.66 104.14) (xy 203.2 104.14))
+    (stroke (width 0) (type default) (color 0 0 0 0))
+  )
+  (wire (pts (xy 219.71 104.14) (xy 222.25 104.14))
+    (stroke (width 0) (type default) (color 0 0 0 0))
+  )
   (wire (pts (xy 92.71 63.5) (xy 107.95 63.5))
     (stroke (width 0) (type default) (color 0 0 0 0))
@@
     (stroke (width 0) (type default) (color 0 0 0 0))
   )
+  (wire (pts (xy 218.44 104.14) (xy 219.71 104.14))
+    (stroke (width 0) (type default) (color 0 0 0 0))
+  )
+  (wire (pts (xy 219.71 104.14) (xy 219.71 80.01))
+    (stroke (width 0) (type default) (color 0 0 0 0))
+  )
   (wire (pts (xy 113.03 71.12) (xy 113.03 74.93))
     (stroke (width 0) (type default) (color 0 0 0 0))
@@
     (stroke (width 0) (type default) (color 0 0 0 0))
   )
+  (wire (pts (xy 161.29 104.14) (xy 161.29 93.98))
+    (stroke (width 0) (type default) (color 0 0 0 0))
+  )
   (wire (pts (xy 102.87 101.6) (xy 102.87 105.41))
     (stroke (width 0) (type default) (color 0 0 0 0))
@@
     (stroke (width 0) (type default) (color 0 0 0 0))
   )
+  (wire (pts (xy 226.06 104.14) (xy 226.06 93.98))
+    (stroke (width 0) (type default) (color 0 0 0 0))
+  )
   (wire (pts (xy 190.5 68.58) (xy 214.63 68.58))
     (stroke (width 0) (type default) (color 0 0 0 0))
@@
     (stroke (width 0) (type default) (color 0 0 0 0))
   )
+  (wire (pts (xy 157.48 104.14) (xy 161.29 104.14))
+    (stroke (width 0) (type default) (color 0 0 0 0))
+  )
   (wire (pts (xy 45.72 123.19) (xy 45.72 68.58))
     (stroke (width 0) (type default) (color 0 0 0 0))
@@
     (stroke (width 0) (type default) (color 0 0 0 0))
   )
-  (wire (pts (xy 200.66 104.14) (xy 203.2 104.14))
-    (stroke (width 0) (type default) (color 0 0 0 0))
-  )
