File: esc_v3_c1/ESC1.kicad_sch (KiCad schematic)
At the start: 39 parts, among them J1 Power, J2 Inputs, J3 Output, Q1 IRF4905, Q10 S8050, Q11 S8050, Q12 S8050, Q2 IRF4905, Q3 IRF4905, Q4 S8050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

Commit message: merge.. but the right thing
Parts:
- J1: footprint Connector_JST:JST_XH_B2B-XH-AM_1x02_P2.50mm_Vertical -> Connector_JST:JST_XH_B2B-XH-A_1x02_P2.50mm_Vertical
Connections:
- net at D6.2 (A), Q12.1 (E): no longer Q9.1 (G)
- net at D5.2 (A), Q11.1 (E): no longer Q8.1 (G)
- net at Q12.3 (C), R9.1: now also Q9.1 (G)
- net at Q11.3 (C), R8.1: now also Q8.1 (G)
- net at D4.2 (A), Q10.1 (E): no longer Q7.1 (G)
- net at Q10.3 (C), R7.1: now also Q7.1 (G)
