File: esc_v3_c1/ESC1.kicad_pcb (KiCad board)
At the start: 2 copper layers, 39 parts, among them J1 Power, J2 Inputs, J3 Output, Q1 IRF4905, Q10 S8050, Q11 S8050, Q12 S8050, Q2 IRF4905, Q3 IRF4905, Q4 S8050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

Commit message: add plot files
Parts:
- J1: footprint Connector_JST:JST_XH_B2B-XH-AM_1x02_P2.50mm_Vertical -> Connector_JST:JST_XH_B2B-XH-A_1x02_P2.50mm_Vertical
- moved Q3 21.1 mm to (119.9, 53.9)
- moved Q9 21.1 mm to (140.2, 53.9)
- moved D10 21.1 mm to (67.1, 49.9)
- moved D11 21.1 mm to (102.4, 49.9)
- moved D2 21.1 mm to (81.8, 26.0)
- moved D4 21.1 mm to (64.0, 26.0)
- moved D5 21.1 mm to (99.6, 26.0)
- moved D6 21.1 mm to (135.1, 26.0)
- moved D8 21.1 mm to (78.1, 49.9)
- moved J3 21.1 mm to (145.8, 33.6)
- moved Q11 21.1 mm to (101.6, 39.6)
- moved Q12 21.1 mm to (137.7, 39.7)
- moved Q5 21.1 mm to (81.8, 39.6)
- moved Q7 21.1 mm to (69.1, 53.6)
- moved Q8 21.1 mm to (104.6, 53.6)
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Routing:
- net VCC: track 261.3 -> 265.5 mm
- net Net-(D12-Pad1): track 84.6 -> 81.6 mm
- net Net-(D10-Pad1): track 184.6 -> 182.4 mm
- net Net-(D11-Pad1): track 136.8 -> 135.0 mm
- net GND: track 13.9 -> 13.0 mm
Other:
- board outline added: 142.2 x 61 mm
- board text added: "A"
- board text added: "A+"
- board text added: "A-"
- board text added: "B"
- board text added: "B+"
- board text added: "B-"
- board text added: "C"
- board text added: "C+"
- board text added: "C-"
- board text added: "ESC Board 3 ©2022 Andrew Woodward-May"
- board text added: "GND"
- board text added: "VCC"
